Commit message: separate odometry

File: ros2_ws/src/common/racecar_description/urdf/racecar.urdf.xacro (robot description, xacro)
@@ -96,5 +96,5 @@
        measured in rad/s. -->
   <xacro:property name="servo_stall_torque" value="0.5649"/>
-  <xacro:property name="servo_no_load_speed" value="4.553"/>
+  <xacro:property name="servo_no_load_speed" value="6.0"/>
   <xacro:property name="dummy_inertia" value="1e-09"/>
   <material name="blue">
@@ -501,5 +501,5 @@
       <right_steering_joint>right_steering_joint</right_steering_joint>
       <wheel_base>${wheelbase}</wheel_base> <!-- Replace with actual value -->
-      <track_width>${hex_hub_dist}</track_width> <!-- Replace with actual value -->
+      <track_width>${hex_hub_dist - 2 * axle_length}</track_width> <!-- Replace with actual value -->
       <wheel_radius>${tire_dia / 2}</wheel_radius> <!-- Replace with actual value -->
       <vel_p_gain>1.0</vel_p_gain>
@@ -511,7 +511,7 @@
       <vel_cmd_min>-10000.0</vel_cmd_min>
       <vel_cmd_offset>0.0</vel_cmd_offset>
-      <steer_p_gain>4.0</steer_p_gain>
+      <steer_p_gain>100.0</steer_p_gain>
       <steer_i_gain>0.1</steer_i_gain>
-      <steer_d_gain>1.0</steer_d_gain>
+      <steer_d_gain>0.1</steer_d_gain>
       <steer_i_max>1.0</steer_i_max>
       <steer_i_min>-1.0</steer_i_min>
@@ -526,66 +526,4 @@
       <steer_topic>steering/position/command</steer_topic> <!-- Replace with actual topic name -->
     </plugin>
-    <!-- <plugin
-      filename="libSpringSystem.so"
-      name="racecar_gazebo::SpringSystem">
-      <spring_constant>1200.0</spring_constant>
-      <damping_constant>150.0</damping_constant>
-      <joint_name>left_front_shock</joint_name>
-      <joint_name>right_front_shock</joint_name>
-      <joint_name>left_rear_shock</joint_name>
-      <joint_name>right_rear_shock</joint_name>
-    </plugin> -->
-    <!-- <plugin
-      filename="gz-sim-joint-controller-system"
-      name="gz::sim::systems::JointController">
-      <joint_name>left_rear_axle</joint_name>
-      <use_force_commands>true</use_force_commands>
-      <topic>left_rear_axle_ctrlr/command</topic>
-      <p_gain>1.5</p_gain>
-      <i_gain>1.0</i_gain>
-      <d_gain>0.0</d_gain>
-      <i_max>10.0</i_max>
-      <i_min>-10.0</i_min>
-    </plugin> -->
-    <!-- <plugin name="gz::sim::systems::AckermannSteering" filename="gz-sim-ackermann-steering-system">
-      <left_joint>left_rear_axle</left_joint>
-      <left_joint>left_front_axle</left_joint>
-      <right_joint>right_rear_axle</right_joint>
-      <right_joint>right_front_axle</right_joint>
-      <left_steering_joint>left_steering_joint</left_steering_joint>
-      <right_steering_joint>right_steering_joint</right_steering_joint>
-      <wheel_separation>${hex_hub_dist}</wheel_separation>
-      <kingpin_width>${axle_length}</kingpin_width>
-      <wheel_base>${wheelbase}</wheel_base>
-      <steering_limit>${degrees_45}</steering_limit>
-      <wheel_radius>${tire_dia / 2}</wheel_radius>
-      <odom_publish_frequency>50</odom_publish_frequency>
-      <min_velocity>-${axle_vel_limit * tire_dia / 2}</min_velocity>
-      <max_velocity>${axle_vel_limit * tire_dia / 2}</max_velocity>
-      <min_acceleration>-50</min_acceleration>
-      <max_acceleration>50</max_acceleration>
-      <min_jerk>-20</min_jerk>
-      <max_jerk>20</max_jerk>
-      <topic>/cmd_vel</topic>
-      <odom_topic>/odom</odom_topic>
-      <tf_topic>tf</tf_topic>
-      <frame_id>odom</frame_id>
-      <child_frame_id>base_link</child_frame_id>
-    </plugin> -->
   </gazebo>
-  <!-- <ros2_control name="GazeboSimSystem" type="system">
-    <hardware>
-      <plugin>gz_ros2_control/GazeboSimSystem</plugin>
-    </hardware>
-    <xacro:shock_trans lr_prefix="left" fr_prefix="front"/>
-    <xacro:shock_trans lr_prefix="right" fr_prefix="front"/>
-    <xacro:shock_trans lr_prefix="left" fr_prefix="rear"/>
-    <xacro:shock_trans lr_prefix="right" fr_prefix="rear"/>
-    <xacro:wheel_trans lr_prefix="left" fr_prefix="front"/>
-    <xacro:wheel_trans lr_prefix="right" fr_prefix="front"/>
-    <xacro:wheel_trans lr_prefix="left" fr_prefix="rear"/>
-    <xacro:wheel_trans lr_prefix="right" fr_prefix="rear"/>
-    <xacro:steering_trans lr_prefix="left"/>
-    <xacro:steering_trans lr_prefix="right"/>
-  </ros2_control> -->
 </robot>

Commit message: Added collision detector

File: ros2_ws/src/common/racecar_description/urdf/racecar.urdf.xacro (robot description, xacro)
@@ -422,5 +422,5 @@
       <material name="gray"/>
     </visual>
-    <collision>
+    <collision name="chassis_collision">
       <origin xyz="0 0 ${-chassis_height / 2}"/>
       <geometry>
@@ -436,4 +436,12 @@
   <gazebo reference="chassis">
     <material>Gazebo/Grey</material>
+    <sensor name='sensor_contact' type='contact'>
+      <contact>
+        <collision>chassis_collision</collision>
+        <topic>/collisions</topic>
+      </contact>
+      <always_on>1</always_on>
+      <update_rate>100</update_rate>
+    </sensor>
   </gazebo>
   <joint name="base_link_to_chasis" type="fixed">
@@ -493,4 +501,8 @@
       <topic>joint_states</topic>
     </plugin>
+    <plugin
+      filename="gz-sim-contact-system"
+      name="gz::sim::systems::Contact">
+    </plugin>
     <plugin name="racecar_gazebo::RacecarController" filename="libRacecarController.so">
       <left_front_wheel_joint>left_front_axle</left_front_wheel_joint>

Commit message: Robot system

File: ros2_ws/src/common/racecar_description/urdf/racecar.urdf.xacro (robot description, xacro)
@@ -33,7 +33,7 @@
   <!-- chassis_length is measured along the x axis, chassis_width
        along the y axis, and chassis_height along the z axis. -->
-  <xacro:property name="chassis_length" value="0.680"/>
-  <xacro:property name="chassis_width" value="0.160"/>
-  <xacro:property name="chassis_height" value="0.01"/>
+  <xacro:property name="chassis_length" value="0.5"/>
+  <xacro:property name="chassis_width" value="0.173"/>
+  <xacro:property name="chassis_height" value="0.06"/>
   <xacro:property name="chassis_mass" value="2.788"/>
   <!-- battery_dist is the distance between the inner edges of the
@@ -58,7 +58,7 @@
   <!--xacro:property name="tire_width" value="0.0889"/-->
   <!--xacro:property name="hex_hub_depth" value="0.01445"/-->
-  <xacro:property name="hub_dia" value="0.102"/>
-  <xacro:property name="tire_dia" value="0.138"/>
-  <xacro:property name="tire_width" value="0.06"/>
+  <xacro:property name="hub_dia" value="0.061"/>
+  <xacro:property name="tire_dia" value="0.1013"/>
+  <xacro:property name="tire_width" value="0.0431"/>
   <xacro:property name="hex_hub_depth" value="0.0"/>
   <xacro:property name="wheel_mass" value="0.29"/>
@@ -67,8 +67,8 @@
        from a U joint to the corresponding hex hub. wheel_travel is the
        vertical wheel travel. -->
-  <xacro:property name="wheelbase" value="0.356"/>
-  <xacro:property name="hex_hub_dist" value="0.385"/>
-  <xacro:property name="axle_length" value="0.03"/>
-  <xacro:property name="wheel_travel" value="0.084"/>
+  <xacro:property name="wheelbase" value="0.320"/>
+  <xacro:property name="hex_hub_dist" value="0.34"/>
+  <xacro:property name="axle_length" value="0.02"/>
+  <xacro:property name="wheel_travel" value="0.042"/>
   <xacro:property name="shock_z_offset" value="0.07"/>
   <!-- shock_eff_limit is 2 * ((shock_stroke / 2) * shock_spring_constant) N.
@@ -400,5 +400,5 @@
   </gazebo>
   <joint name="imu_joint" type="fixed">
-    <origin xyz="0 0 0.008" rpy="0 0 0" />
+    <origin xyz="-0.07 0 0.0095" rpy="0 ${degrees_90 * 2} 0" />
     <parent link="chassis" />
     <child link="imu_link" />
@@ -485,7 +485,4 @@
   </gazebo> -->
   <gazebo>
-    <!-- <plugin filename="libgz_ros2_control-system.so" name="gz_ros2_control::GazeboSimROS2ControlPlugin">
-      <parameters>$(find racecar_gazebo)/config/control_params.yaml</parameters>
-    </plugin> -->
     <plugin
       filename="gz-sim-joint-state-publisher-system"
