Commit message: Change simulator to gym

File: ros2_ws/src/common/racecar_description/urdf/accessories.urdf.xacro (robot description, xacro)
@@ -2,5 +2,5 @@
 <robot xmlns:xacro="http://ros.org/wiki/xacro">
   <xacro:include filename="$(find racecar_description)/urdf/accessories/hokuyo_ust10.urdf.xacro" />
-  <xacro:hokuyo_ust10_mount prefix="front" topic="scan" parent_link="chassis">
+  <xacro:hokuyo_ust10_mount prefix="${robot_prefix}front" topic="scan" parent_link="${robot_prefix}chassis">
     <origin xyz="0.2425 0.00 0.07" rpy="0 0 0" />
   </xacro:hokuyo_ust10_mount>

File: ros2_ws/src/common/racecar_description/urdf/racecar.urdf.xacro (robot description, xacro)
@@ -28,4 +28,7 @@
 -->
 <robot name="racecar" xmlns:xacro="http://www.ros.org/wiki/xacro">
+  <!-- Argument prefix -->
+  <xacro:arg name="robot_prefix" default=""/>
+  <xacro:property name="robot_prefix" value="$(arg robot_prefix)"/>
   <!-- Degree-to-radian conversions -->
   <xacro:property name="degrees_45" value="0.785398163"/>
@@ -154,7 +157,7 @@
   <!-- Battery -->
   <xacro:macro name="battery" params="prefix reflect">
-    <joint name="chassis_to_${prefix}_battery" type="fixed">
-      <parent link="chassis"/>
-      <child link="${prefix}_battery_offset"/>
+    <joint name="${robot_prefix}chassis_to_${prefix}_battery" type="fixed">
+      <parent link="${robot_prefix}chassis"/>
+      <child link="${robot_prefix}${prefix}_battery_offset"/>
       <origin xyz="${battery_x_offset - battery_length / 2}
                    ${reflect * battery_dist / 2}
@@ -162,15 +165,15 @@
               rpy="${reflect * battery_comp_angle} 0 0"/>
     </joint>
-    <link name="${prefix}_battery_offset">
+    <link name="${robot_prefix}${prefix}_battery_offset">
       <xacro:null_inertial/>
     </link>
-    <joint name="offset_to_${prefix}_battery" type="fixed">
-      <parent link="${prefix}_battery_offset"/>
-      <child link="${prefix}_battery"/>
+    <joint name="${robot_prefix}offset_to_${prefix}_battery" type="fixed">
+      <parent link="${robot_prefix}${prefix}_battery_offset"/>
+      <child link="${robot_prefix}${prefix}_battery"/>
       <origin xyz="0
                    ${reflect * battery_width / 2}
                    ${(battery_height / 2) - battery_comp_depth}"/>
     </joint>
-    <link name="${prefix}_battery">
+    <link name="${robot_prefix}${prefix}_battery">
       <visual>
         <geometry>
@@ -190,5 +193,5 @@
       </xacro:solid_cuboid_inertial>
     </link>
-    <gazebo reference="${prefix}_battery">
+    <gazebo reference="${robot_prefix}${prefix}_battery">
       <material>Gazebo/Blue</material>
     </gazebo>
@@ -197,8 +200,8 @@
   <xacro:macro name="shock"
                params="lr_prefix fr_prefix lr_reflect fr_reflect child">
-    <joint name="${lr_prefix}_${fr_prefix}_shock" type="prismatic">
-    <!-- <joint name="${lr_prefix}_${fr_prefix}_shock" type="fixed"> -->
-      <parent link="chassis"/>
-      <child link="${child}"/>
+    <joint name="${robot_prefix}${lr_prefix}_${fr_prefix}_shock" type="prismatic">
+    <!-- <joint name="${robot_prefix}${lr_prefix}_${fr_prefix}_shock" type="fixed"> -->
+      <parent link="${robot_prefix}chassis"/>
+      <child link="${robot_prefix}${child}"/>
       <origin xyz="${fr_reflect * wheelbase / 2}
                    ${lr_reflect * ((hex_hub_dist / 2) - axle_length)}
@@ -209,5 +212,5 @@
              effort="${shock_eff_limit}" velocity="${shock_vel_limit}"/>
     </joint>
-    <gazebo reference="${lr_prefix}_${fr_prefix}_shock">
+    <gazebo reference="${robot_prefix}${lr_prefix}_${fr_prefix}_shock">
       <implicitSpringDamper>true</implicitSpringDamper>
       <springStiffness>10000</springStiffness>
@@ -216,5 +219,5 @@
   </xacro:macro>
   <xacro:macro name="shock_trans" params="lr_prefix fr_prefix">
-    <joint name="${lr_prefix}_${fr_prefix}_shock">
+    <joint name="${robot_prefix}${lr_prefix}_${fr_prefix}_shock">
       <command_interface name="effort">
         <param name="min">-${shock_eff_limit}</param>
@@ -234,12 +237,12 @@
   <!-- The "wheel" macro defines an axle carrier, axle, and wheel. -->
   <xacro:macro name="wheel" params="lr_prefix fr_prefix lr_reflect">
-    <link name="${lr_prefix}_${fr_prefix}_axle_carrier">
+    <link name="${robot_prefix}${lr_prefix}_${fr_prefix}_axle_carrier">
       <xacro:null_inertial/>
     </link>
     <!-- The left and right axles have the same axis so that identical
          rotation values cause the wheels to rotate in the same direction. -->
-    <joint name="${lr_prefix}_${fr_prefix}_axle" type="continuous">
-      <parent link="${lr_prefix}_${fr_prefix}_axle_carrier"/>
-      <child link="${lr_prefix}_${fr_prefix}_wheel"/>
+    <joint name="${robot_prefix}${lr_prefix}_${fr_prefix}_axle" type="continuous">
+      <parent link="${robot_prefix}${lr_prefix}_${fr_prefix}_axle_carrier"/>
+      <child link="${robot_prefix}${lr_prefix}_${fr_prefix}_wheel"/>
       <origin rpy="${degrees_90} 0 0"/>
       <axis xyz="0 0 -1"/>
@@ -249,5 +252,5 @@
     <!-- <transmission name="${lr_prefix}_${fr_prefix}_axle_trans">
       <type>transmission_interface/SimpleTransmission</type>
-      <joint name="${lr_prefix}_${fr_prefix}_axle">
+      <joint name="${robot_prefix}${lr_prefix}_${fr_prefix}_axle">
         <hardwareInterface>hardware_interface/EffortJointInterface</hardwareInterface>
       </joint>
@@ -257,5 +260,5 @@
       </actuator>
     </transmission> -->
-    <link name="${lr_prefix}_${fr_prefix}_wheel">
+    <link name="${robot_prefix}${lr_prefix}_${fr_prefix}_wheel">
       <visual>
         <origin xyz="0
@@ -281,5 +284,5 @@
           height="${tire_width}" mass="${wheel_mass}"/>
     </link>
-    <gazebo reference="${lr_prefix}_${fr_prefix}_wheel">
+    <gazebo reference="${robot_prefix}${lr_prefix}_${fr_prefix}_wheel">
       <material>Gazebo/Black</material>
       <selfCollide>false</selfCollide>
@@ -306,5 +309,5 @@
   </xacro:macro>
   <xacro:macro name="wheel_trans" params="lr_prefix fr_prefix">
-    <joint name="${lr_prefix}_${fr_prefix}_axle">
+    <joint name="${robot_prefix}${lr_prefix}_${fr_prefix}_axle">
       <!-- <command_interface name="effort"> -->
       <state_interface name="effort">
@@ -329,10 +332,10 @@
                  lr_reflect="${lr_reflect}" fr_reflect="${fr_reflect}"
                  child="${lr_prefix}_steering_link"/>
-    <link name="${lr_prefix}_steering_link">
+    <link name="${robot_prefix}${lr_prefix}_steering_link">
       <xacro:null_inertial/>
     </link>
-    <joint name="${lr_prefix}_steering_joint" type="revolute">
-      <parent link="${lr_prefix}_steering_link"/>
-      <child link="${lr_prefix}_${fr_prefix}_axle_carrier"/>
+    <joint name="${robot_prefix}${lr_prefix}_steering_joint" type="revolute">
+      <parent link="${robot_prefix}${lr_prefix}_steering_link"/>
+      <child link="${robot_prefix}${lr_prefix}_${fr_prefix}_axle_carrier"/>
       <axis xyz="0 0 1"/>
       <dynamics damping="0.2" />
@@ -340,5 +343,5 @@
              effort="${servo_stall_torque}" velocity="${servo_no_load_speed}"/>
     </joint>
-    <gazebo reference="${lr_prefix}_steering_joint">
+    <gazebo reference="${robot_prefix}${lr_prefix}_steering_joint">
       <selfCollide>false</selfCollide>
       <mu1 value="1.5"/>
@@ -350,5 +353,5 @@
     <!-- <transmission name="${lr_prefix}_steering_trans">
       <type>transmission_interface/SimpleTransmission</type>
-      <joint name="${lr_prefix}_steering_joint">
+      <joint name="${robot_prefix}${lr_prefix}_steering_joint">
         <hardwareInterface>hardware_interface/EffortJointInterface</hardwareInterface>
       </joint>
@@ -362,5 +365,5 @@
   </xacro:macro>
   <xacro:macro name="steering_trans" params="lr_prefix">
-    <joint name="${lr_prefix}_steering_joint">
+    <joint name="${robot_prefix}${lr_prefix}_steering_joint">
       <command_interface name="effort">
         <param name="min">-${servo_stall_torque}</param>
@@ -388,5 +391,5 @@
   <!-- base_link must have geometry so that its axes can be displayed in
        rviz. -->
-  <link name="base_link">
+  <link name="${robot_prefix}base_link">
     <visual>
       <geometry>
@@ -396,13 +399,13 @@
     </visual>
   </link>
-  <gazebo reference="base_link">
+  <gazebo reference="${robot_prefix}base_link">
     <material>Gazebo/Grey</material>
   </gazebo>
-  <joint name="imu_joint" type="fixed">
+  <joint name="${robot_prefix}imu_joint" type="fixed">
     <origin xyz="-0.07 0 0.0095" rpy="0 ${degrees_90 * 2} 0" />
-    <parent link="chassis" />
-    <child link="imu_link" />
+    <parent link="${robot_prefix}chassis" />
+    <child link="${robot_prefix}imu_link" />
   </joint>
-  <link name="imu_link">
+  <link name="${robot_prefix}imu_link">
     <inertial>
       <origin xyz="0 0 0" rpy="0 0 0" />
@@ -414,5 +417,5 @@
   </link>
   <!-- Chassis -->
-  <link name="chassis">
+  <link name="${robot_prefix}chassis">
     <visual>
       <origin xyz="0 0 ${-chassis_height / 2}"/>
@@ -434,5 +437,5 @@
     </xacro:solid_cuboid_inertial>
   </link>
-  <gazebo reference="chassis">
+  <gazebo reference="${robot_prefix}chassis">
     <material>Gazebo/Grey</material>
     <sensor name='sensor_contact' type='contact'>
@@ -445,7 +448,7 @@
     </sensor>
   </gazebo>
-  <joint name="base_link_to_chasis" type="fixed">
-    <parent link="base_link"/>
-    <child link="chassis"/>
+  <joint name="${robot_prefix}base_link_to_chasis" type="fixed">
+    <parent link="${robot_prefix}base_link"/>
+    <child link="${robot_prefix}chassis"/>
   </joint>
   <!-- Batteries -->
@@ -468,5 +471,5 @@
     </plugin>
   </gazebo>
-  <gazebo reference="imu_link">
+  <gazebo reference="${robot_prefix}imu_link">
     <sensor name="imu_sensor" type="imu">
       <topic>imu/data</topic>
@@ -503,10 +506,10 @@
     </plugin>
     <plugin name="racecar_gazebo::RacecarController" filename="libRacecarController.so">
-      <left_front_wheel_joint>left_front_axle</left_front_wheel_joint>
-      <right_front_wheel_joint>right_front_axle</right_front_wheel_joint>
-      <left_rear_wheel_joint>left_rear_axle</left_rear_wheel_joint>
-      <right_rear_wheel_joint>right_rear_axle</right_rear_wheel_joint>
-      <left_steering_joint>left_steering_joint</left_steering_joint>
-      <right_steering_joint>right_steering_joint</right_steering_joint>
+      <left_front_wheel_joint>${robot_prefix}left_front_axle</left_front_wheel_joint>
+      <right_front_wheel_joint>${robot_prefix}right_front_axle</right_front_wheel_joint>
+      <left_rear_wheel_joint>${robot_prefix}left_rear_axle</left_rear_wheel_joint>
+      <right_rear_wheel_joint>${robot_prefix}right_rear_axle</right_rear_wheel_joint>
+      <left_steering_joint>${robot_prefix}left_steering_joint</left_steering_joint>
+      <right_steering_joint>${robot_prefix}right_steering_joint</right_steering_joint>
       <wheel_base>${wheelbase}</wheel_base> <!-- Replace with actual value -->
       <track_width>${hex_hub_dist - 2 * axle_length}</track_width> <!-- Replace with actual value -->

Commit message: Added pure pursuit and static planner

File: ros2_ws/src/common/racecar_description/urdf/accessories.urdf.xacro (robot description, xacro)
@@ -3,5 +3,5 @@
   <xacro:include filename="$(find racecar_description)/urdf/accessories/hokuyo_ust10.urdf.xacro" />
   <xacro:hokuyo_ust10_mount prefix="${robot_prefix}front" topic="scan" parent_link="${robot_prefix}chassis">
-    <origin xyz="0.2425 0.00 0.07" rpy="0 0 0" />
+    <origin xyz="0.15 0.00 0.07" rpy="0 0 0" />
   </xacro:hokuyo_ust10_mount>
 </robot>
